File: board/nixieclockboard.kicad_pcb (KiCad board)
At the start: 2 copper layers, 70 x 65 mm, 90 parts, among them IC1 ATMEGA328P-A, P1 PWR, P10 ANODE, P11 5V, P12 5V, P13 ADC, P2 BUZZ, P3 HVSUP, P4 5V, P5 BTN, P6 ISP, P7 SERIAL, P8 I2C, P9 D0, Q1 2N7000, Q10 MPSA42, Q11 MPSA42, Q12 MPSA42, Q13 MPSA42, Q14 MPSA42, Q15 MPSA42, Q16 IRF740, Q17 BC547, Q2 MPSA92, Q3 MPSA92, Q4 MPSA92, Q5 MPSA92, Q6 MPSA92, Q7 MPSA92, Q8 MPSA42, Q9 MPSA42, U1 LM1117, U2 K155ID1, U3 555, X1 18.432MHz

Commit message: Board completed
Parts:
- removed P3: HVSUP, PA_1X3
- added R5: 10k, SM0805, B.Cu at (213.0, 160.5)
- added SCREW_M3: VAL**, SCREW_M3, F.Cu at (163.0, 123.0)
- added SCREW_M3: VAL**, SCREW_M3, F.Cu at (227.0, 123.0)
- added SCREW_M3: VAL**, SCREW_M3, F.Cu at (227.0, 162.0)
- added SCREW_M3: VAL**, SCREW_M3, F.Cu at (163.0, 162.0)
- C4, C5: footprint CPE_5mm -> SM1206POL; moved to B.Cu
- R21, R22, R23, R24, R25, R26: value 8k2 -> R
- U1: footprint SOT223 -> SOT223-LM1117
- moved P12 52.1 mm to (190.7, 160.5)
- moved P13 47.7 mm to (202.7, 150.9), turned to 90 degrees
- moved C1 29.2 mm to (219.9, 156.2), turned to 0 degrees
- moved P8 28.0 mm to (210.5, 142.0), turned to 90 degrees
- moved P5 27.8 mm to (225.0, 137.5), turned to 270 degrees
- moved P2 26.2 mm to (203.2, 163.0), turned to 180 degrees
- moved JP1 25.3 mm to (200.7, 160.8), turned to 0 degrees
- moved P4 23.1 mm to (219.2, 160.3), turned to 180 degrees
- moved P11 21.2 mm to (219.2, 162.8), turned to 180 degrees
- moved C2 20.9 mm to (222.0, 139.5)
- moved P7 18.7 mm to (215.5, 142.0), turned to 90 degrees
- moved C3 18.5 mm to (222.0, 141.5), turned to 180 degrees
- moved R9 17.3 mm to (199.2, 147.5), turned to 180 degrees
- moved R1 17.2 mm to (208.1, 147.4), turned to 0 degrees
- moved R7 16.8 mm to (199.2, 145.6)
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Connections:
- net N-0000065 renamed /BUZ-
- net N-0000075 renamed /BUZ+
- C4 pad 1: /VSUP -> /HVSupply/VIN
- JP1 pad 1: /VSUP -> /HVSupply/VIN
- P1 pad 2: /VSUP -> /HVSupply/VIN
- P7 pad 1: /TXD -> /RXD
- P7 pad 2: /RXD -> /TXD
- Q2 pad 1: /AE0 -> HV
- Q2 pad 3: HV -> /AE0
- Q3 pad 1: /AE1 -> HV
- Q3 pad 3: HV -> /AE1
- Q4 pad 1: /AE2 -> HV
- Q4 pad 3: HV -> /AE2
- Q5 pad 1: /AE3 -> HV
- Q5 pad 3: HV -> /AE3
- Q6 pad 1: /AE4 -> HV
- Q6 pad 3: HV -> /AE4
- Q7 pad 1: /AE5 -> HV
- Q7 pad 3: HV -> /AE5
- U1 pad 3: /VSUP -> /HVSupply/VIN
Routing:
- net /HVSupply/VIN: track 27.4 -> 90.5 mm
- net GND: track 9.79 -> 70.0 mm, vias 6 -> 11
- net /VSUP: track 55.7 -> 0.00 mm, vias 1 -> 0
- net /HVSupply/VPUMP: track 0.00 -> 34.4 mm
- net /VCC: track 0.00 -> 19.4 mm, vias 0 -> 4
- net HV: track 95.6 -> 79.8 mm
- net /BIT0: track 16.5 -> 30.1 mm, vias 0 -> 1
- net /ADC7: track 0.00 -> 12.6 mm
- net /HVSupply/TRG: track 11.7 -> 23.7 mm
- net /BUZZ: track 18.3 -> 7.87 mm
- net /ADC6: track 1.95 -> 12.1 mm
- net /BALARM: track 3.61 -> 13.1 mm
- net /BZONE: track 3.55 -> 12.6 mm
- net /HVSupply/NPNC: track 3.50 -> 12.1 mm, vias 0 -> 1
- net /BIT2: track 22.0 -> 29.2 mm
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- added copper zone on B.Cu, net /HVSupply/VIN
Other:
- board size 70 x 65 mm -> 70 x 45 mm
- board text added: "(A)"
- board text added: "(B)"
- board text added: "ANODE RESISTORS 10k - 20k"
- board text added: "NIXIEBOARD G ROBINSON 2015"
- board text added: "REVISION NOTES V2 2015-03-19 (A) R21-R26 WERE 8K2 (B) U1 P4 WAS N/C"
- board text added: "V2"

Commit message: Add board design
Parts:
- added G***: LOGO, george:grlogo_05mm, F.Cu at (177.0, 182.0)
- C1, C10, C11, C2, C3, C6, C7: footprint SM0805 -> Capacitors_SMD:C_0805
- C4, C5: footprint SM1206POL -> Capacitors_SMD:C_1206
- C8: footprint CPE_8mm -> Capacitors_THT:CP_Radial_D8.0mm_P3.80mm
- C9: footprint CPE_10mm -> Capacitors_THT:CP_Radial_D10.0mm_P5.00mm
- D1, D2: footprint D4 -> Diodes_THT:D_DO-35_SOD27_P7.62mm_Horizontal
- IC1: footprint TQFP32 -> Housings_QFP:TQFP-32_7x7mm_Pitch0.8mm
- JP1, JP2, JP3: footprint JUMPER_SMD -> george:JUMPER_SMD_3
- L1: footprint IND_R_10 -> Inductors_THT:L_Radial_D10.0mm_P5.00mm_Fastron_07M
- P1, P11, P12, P13, P2, P4, P7, P8: footprint PA_1X2 -> Pin_Headers:Pin_Header_Straight_1x02_Pitch2.54mm
- P10: footprint PA_1X6 -> Pin_Headers:Pin_Header_Straight_1x06_Pitch2.54mm
- P5: footprint PA_1X4 -> Pin_Headers:Pin_Header_Straight_1x04_Pitch2.54mm
- P6: footprint PA_2X3 -> Pin_Headers:Pin_Header_Straight_2x03_Pitch2.54mm
- P9: footprint PA_1X12 -> Pin_Headers:Pin_Header_Straight_1x12_Pitch2.54mm
- Q1: footprint TO92DGS -> TO_SOT_Packages_THT:TO-92_Molded_Narrow
- Q10, Q11, Q12, Q13, Q14, Q15, Q2, Q3, Q4, Q5, Q6, Q7, Q8, Q9: footprint TO92-S-123 -> TO_SOT_Packages_THT:TO-92_Molded_Narrow
- Q16: footprint TO220_VERT_GDS -> TO_SOT_Packages_THT:TO-220_Vertical
- Q17: footprint TO92-S-321 -> TO_SOT_Packages_THT:TO-92_Molded_Narrow
- R1, R10, R11, R12, R13, R14, R15, R16, R17, R18, R19, R2, R20, R21, R22, R23, R24, R25, R26, R27, R28, R29, R3, R30, R31, R32, R33, R34, R35, R36, R37, R38, R4, R5, R6, R7, R8, R9: footprint SM0805 -> Resistors_SMD:R_0805
- RV1: footprint POT_CERMET_VERT -> Potentiometers:Potentiometer_Trimmer_Bourns_PV36W
- U1: footprint SOT223-LM1117 -> TO_SOT_Packages_SMD:SOT-223-3Lead_TabPin2
- U2: footprint DIP-16__300 -> Housings_DIP:DIP-16_W7.62mm
- U3: footprint so-8 -> Housings_SOIC:SO-8_5.3x6.2mm_Pitch1.27mm
- X1: footprint CRYSTAL -> Crystals:Crystal_HC49-4H_Vertical
- moved U2 9.81 mm to (199.0, 134.4), turned to 90 degrees
- moved D2 5.10 mm to (186.1, 153.0)
- moved C9 2.60 mm to (179.5, 153.6), turned to 90 degrees
- moved Q16 2.60 mm to (174.4, 160.6), turned to 180 degrees
- moved D1 2.50 mm to (207.5, 129.6)
- moved L1 2.50 mm to (168.5, 149.8)
- moved RV1 2.50 mm to (180.3, 160.1)
- moved X1 2.27 mm to (223.5, 149.6)
- moved C8 2.00 mm to (165.5, 141.0)
- moved Q10 1.30 mm to (173.7, 136.5)
- moved Q11 1.30 mm to (179.7, 136.5)
- moved Q12 1.30 mm to (185.7, 136.5)
- moved Q13 1.30 mm to (191.7, 136.5)
- moved Q2 1.30 mm to (161.7, 130.0)
- moved Q3 1.30 mm to (167.7, 130.0)
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Connections:
- net /HVSupply/VIN renamed /VSUP
- IC1 pad 10: /BIT2 -> /BIT1
- IC1 pad 11: /BIT3 -> /BIT0
- IC1 pad 2: /BIT0 -> /BIT3
- IC1 pad 9: /BIT1 -> /BIT2
- P2 pad 1: /BUZ- -> (no net)
- U2 pad 3: /BIT3 -> /BIT0
- U2 pad 4: /BIT0 -> /BIT3
- U2 pad 6: /BIT2 -> /BIT1
- U2 pad 7: /BIT1 -> /BIT2
- U3 pad 3: /HVSupply/OSC -> (no net)
Routing:
- net /HVSupply/OSC: track 19.2 -> 0.00 mm, vias 1 -> 0
- net /HVSupply/DIS: track 5.08 -> 20.8 mm, vias 0 -> 1
- net /BIT0: track 30.1 -> 37.5 mm
- net /BIT3: track 37.5 -> 30.1 mm
- net /VSUP: track 90.5 -> 84.6 mm
- net GND: track 70.0 -> 74.7 mm
- net /BUZ-: track 3.87 -> 0.00 mm
- net (no net): track 0.00 -> 3.87 mm
- net /HVSupply/TRG: track 23.7 -> 27.1 mm
- net /BIT1: track 26.3 -> 29.2 mm
- net /BIT2: track 29.2 -> 26.3 mm
- net /HVSupply/NPNC: track 12.1 -> 13.3 mm
- added copper zone on B.Cu, net /HVSupply/VIN
- removed copper zone on B.Cu, net /VSUP
Other:
- board text added: "NIXIEQUAD REV03 2017-10-03"
- board text added: "REVISION NOTES 03 2017-10-03 PACKAGES UPDATED TO NEW STYLE"
