File: board/nixieclockboard.sch (KiCad schematic (older format))
At the start: 28 parts

Commit message: Schematic updates
Parts:
- removed C?: 0u33, symbol CP1
- removed C?: 0u1, symbol CP1
- removed U?: 7805, symbol 7805
- added C? (x2): 10u, ~, symbol CP1
- added C?: 0u1, ~, symbol C
- added JP?: S4/SD8, ~, symbol JUMPER3
- added JP?: S5/SCL, ~, symbol JUMPER3
- added JP?: S4/RXD, ~, symbol JUMPER3
- added JP?: S4/TXD, ~, symbol JUMPER3
- added K?: A1, symbol CONN_3
- added K?: A2, symbol CONN_3
- added R?: 120, ~, symbol R
- added R?: 360, ~, symbol R
- added R? (x4): R, ~, symbol R
- added R? (x2): 10k, ~, symbol R
Connections:
- net labels added: ADC6, ADC7, ADJ, PC4, PC5, PD0, PD1, SCL, SDA
- wire segments 128 -> 173
Other:
- note added: "5V REGULATOR"
- note added: "ANODE DRIVERS AND HEADERS"
- note added: "BUZZER"
- note added: "COMMA CATHODE DRIVERS"
- note added: "CONFIG JUMPERS\n(6 DIGITS) || (I2C) || (SERIAL)"
- note added: "GENERIC ANALOG"
- note added: "GPS/SERIAL INTERFACE"
- note added: "HV SUPPLY"
- note added: "MICROCONTROLLER"
- note added: "NIXIE CATHODE DRIVER"
- note added: "OSCIALLTOR"
- note added: "POWER INPUT"
- note added: "PROGRAMMER / SPI"
- note removed: "JUMPER P104 'HVSUP':\n2-1: POWER SUPPLIED TO HV\nNC: NO POWER SUPPLIED TO HV"
- moved on the sheet: D?, P?, Q?, U?

Commit message: Schematic and board creation continued
Parts:
- removed JP?: S4/RXD, ~, symbol JUMPER3
- removed JP?: S4/TXD, ~, symbol JUMPER3
- removed K?: A1, symbol CONN_3
- removed K?: A2, symbol CONN_3
- removed R?: 10k, symbol R
- removed U?: GPS, symbol SKM53
- added P10: ANODE, symbol CONN_6
- added P11, P12, P4: 5V, symbol CONN_2
- added P13: ADC, symbol CONN_2
- added P7: SERIAL, symbol CONN_2
- added P8: I2C, symbol CONN_2
- added P9: D0, symbol CONN_12
- added Q10, Q11, Q12, Q13, Q8, Q9: MPSA42, ~, symbol NPN
- added Q2, Q3, Q4, Q5, Q6, Q7: MPSA92, ~, symbol PNP
- added R11, R12, R13, R14, R15, R16: 100k, ~, symbol R
- added R21, R22, R23, R24, R25, R26: 8k2, ~, symbol R
- added R27, R28, R29, R30, R31, R32: 10k, ~, symbol R
- C2: renamed from 0u?; value C -> 0u1
- C3: renamed from 0u1; value C -> 0u1
- JP2: renamed from JP?; value S4/SD8 -> S4/SDA
- P1: renamed from P?; value 12V IN -> PWR
- gave numbers to parts that had none: 32
Connections:
- net labels added: A0, A1, A2, A3, A4, A5, AE0, AE1, AE2, AE3, AE4, AE5, C0, C1, C2, C3, C4, C5, C6, C7, C8, C9, CLB, CLC, CRB, CRC, NPNB0, NPNB1, NPNB2, NPNB3, NPNB4, NPNB5, PNPB0, PNPB1, PNPB2, PNPB3, PNPB4, PNPB5
- net labels removed: CLNPNB, CRNPNB, D0, D1, D2, D3, D4, D5, D6, D7, D8, D9, GR, PC4, PC5, PD0, PD1, XTAL1, XTAL2
- wire segments 173 -> 226
- no-connect marks 1 -> 0
Other:
- note added: "ANODE DRIVERS"
- note added: "POWER OUTPUT"
- note added: "TUBE HEADERS"
- note removed: "ANODE DRIVERS AND HEADERS"
- moved on the sheet: D1, IC1, JP1, JP2, JP3, P1, P2, P5, P6, Q1, Q14, Q15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

Commit message: Board completed
Parts:
- removed P3: HVSUP, symbol CONN_3
- added R5: 10k, ~, symbol R
- R21, R22, R23, R24, R25, R26: value 8k2 -> R
Connections:
- net labels added: BUZ+, BUZ-
- net labels removed: VSUP_SW
- wire segments 226 -> 225
Other:
- note added: "(A)"
- note added: "REVISION NOTES V2 2015-03-19\n(A) R21-R26 WERE 8K2"
- moved on the sheet: JP1, P2, Q1
Changed lines of the file:
@@
 encoding utf-8
 Sheet 1 2
-Title ""
-Date "21 jan 2015"
-Rev ""
+Title "NIXIEBOARD"
+Date "18 mar 2015"
+Rev "V2"
 Comp ""
 Comment1 ""
@@
 Comment4 ""
 $EndDescr
-Connection ~ 12350 3050
-Wire Wire Line
-	5350 3050 5350 3150
+Wire Wire Line
+	5700 2250 5700 2350
 Wire Wire Line
 	3000 8800 2750 8800
@@
 	7150 9700 6950 9700
 Wire Wire Line
-	5050 3350 4900 3350
+	4900 2550 5400 2550
 Wire Wire Line
 	2350 8800 2250 8800
@@
 Connection ~ 2250 9200
 Wire Wire Line
-	5150 3700 5350 3700
-Wire Wire Line
-	5350 3700 5350 3550
-Wire Wire Line
-	14100 2850 13750 2850
-$Comp
-L CONN_3 P3
-U 1 1 4DF9FAE7
-P 14450 2950
-F 0 "P3" V 14400 2950 50  0000 C CNN
-F 1 "HVSUP" V 14500 2950 40  0000 C CNN
-F 2 "" H 14450 2950 60  0001 C CNN
-F 3 "" H 14450 2950 60  0001 C CNN
-	1    14450 2950
-	1    0    0    1
-$EndComp
+	5700 3400 4900 3400
+Wire Wire Line
+	5700 2750 5700 3400
 $Comp
 L MOSFET_N Q1
 U 1 1 4DF56A57
-P 5250 3350
-F 0 "Q1" H 5260 3520 60  0000 R CNN
-F 1 "2N7000" H 5260 3200 60  0000 R CNN
-F 2 "" H 5250 3350 60  0001 C CNN
-F 3 "" H 5250 3350 60  0001 C CNN
-	1    5250 3350
-	1    0    0    -1
-$EndComp
-Text Label 4900 3350 2    60   ~ 0
+P 5600 2550
+F 0 "Q1" H 5610 2720 60  0000 R CNN
+F 1 "2N7000" H 5610 2400 60  0000 R CNN
+F 2 "" H 5600 2550 60  0001 C CNN
+F 3 "" H 5600 2550 60  0001 C CNN
+	1    5600 2550
+	1    0    0    -1
+$EndComp
+Text Label 4900 2550 2    60   ~ 0
 BUZZ
 Text Label 3450 1700 0    60   ~ 0
@@
 VCC
 Text Label 12300 3050 2    60   ~ 0
-VSUP_SW
+VSUP
 $Sheet
-S 12500 2600 550  700
+S 12500 2600 1600 700
 U 4DE4A3C9
 F0 "HVSupply" 60
@@
 CONTROL
 Wire Wire Line
-	5100 2500 4750 2500
-Text Label 4750 2500 0    60   ~ 0
+	5450 1700 5100 1700
+Text Label 5100 1700 0    60   ~ 0
 VSUP
 $Comp
 L CONN_2 P2
 U 1 1 54AFA8EB
-P 5750 2950
-F 0 "P2" V 5700 2950 40  0000 C CNN
-F 1 "BUZZ" V 5800 2950 40  0000 C CNN
-F 2 "" H 5750 2950 60  0000 C CNN
-F 3 "" H 5750 2950 60  0000 C CNN
-	1    5750 2950
+P 6450 2150
+F 0 "P2" V 6400 2150 40  0000 C CNN
+F 1 "BUZZ" V 6500 2150 40  0000 C CNN
+F 2 "" H 6450 2150 60  0000 C CNN
+F 3 "" H 6450 2150 60  0000 C CNN
+	1    6450 2150
 	1    0    0    1
 $EndComp
@@
 L JUMPER3 JP1
 U 1 1 54AFAA5F
-P 5350 2500
-F 0 "JP1" H 5400 2400 40  0000 L CNN
-F 1 "VBUZZ" H 5350 2600 40  0000 C CNN
-F 2 "~" H 5350 2500 60  0000 C CNN
-F 3 "~" H 5350 2500 60  0000 C CNN
-	1    5350 2500
-	1    0    0    -1
-$EndComp
-Wire Wire Line
-	5600 2500 5850 2500
-Text Label 5850 2500 0    60   ~ 0
+P 5700 1700
+F 0 "JP1" H 5750 1600 40  0000 L CNN
+F 1 "VBUZZ" H 5700 1800 40  0000 C CNN
+F 2 "~" H 5700 1700 60  0000 C CNN
+F 3 "~" H 5700 1700 60  0000 C CNN
+	1    5700 1700
+	1    0    0    -1
+$EndComp
+Wire Wire Line
+	5950 1700 6200 1700
+Text Label 6200 1700 0    60   ~ 0
 VCC
 Wire Wire Line
-	5350 2600 5350 2850
+	5700 1800 5700 2050
 $Comp
 L C C3
@@
 	1950 6500 1950 6400
 Wire Wire Line
-	5350 2850 5400 2850
-Wire Wire Line
-	5400 3050 5350 3050
+	5700 2050 6100 2050
+Wire Wire Line
+	5700 2250 6100 2250
 $Comp
 L LM1117 U1
@@
 	0    -1   -1   0
 $EndComp
-Wire Wire Line
-	13750 3050 14100 3050
-Text Label 13750 3050 2    60   ~ 0
-VSUP
-Wire Wire Line
-	14100 2950 13750 2950
-Text Label 13750 2950 2    60   ~ 0
-VSUP_SW
-Text Label 13750 2850 2    60   ~ 0
-GND
 Text Label 6300 10250 1    60   ~ 0
 GND
@@
 Text Notes 5650 8600 0    60   ~ 0
 COMMA CATHODE DRIVERS
-Text Notes 4750 2250 0    60   ~ 0
+Text Notes 5100 1450 0    60   ~ 0
 BUZZER
 Text Notes 3000 5750 0    60   ~ 0
@@
 P 9950 9200
 F 0 "Q2" H 9950 9050 60  0000 R CNN
-F 1 "MPSA92" V 9950 9700 60  0000 R CNN
+F 1 "MPSA92" V 9950 8900 60  0000 R CNN
 F 2 "~" H 9950 9200 60  0000 C CNN
 F 3 "~" H 9950 9200 60  0000 C CNN
 	1    9950 9200
-	1    0    0    -1
+	1    0    0    1
 $EndComp
 $Comp
@@
 P 10050 9800
 F 0 "R21" V 10130 9800 40  0000 C CNN
-F 1 "8k2" V 10057 9801 40  0000 C CNN
+F 1 "R" V 10057 9801 40  0000 C CNN
 F 2 "~" V 9980 9800 30  0000 C CNN
 F 3 "~" H 10050 9800 30  0000 C CNN
@@
 P 11050 9200
 F 0 "Q3" H 11050 9050 60  0000 R CNN
-F 1 "MPSA92" V 11050 9700 60  0000 R CNN
+F 1 "MPSA92" V 11050 8900 60  0000 R CNN
 F 2 "~" H 11050 9200 60  0000 C CNN
 F 3 "~" H 11050 9200 60  0000 C CNN
 	1    11050 9200
-	1    0    0    -1
+	1    0    0    1
 $EndComp
 $Comp
@@
 P 11150 9800
 F 0 "R22" V 11230 9800 40  0000 C CNN
-F 1 "8k2" V 11157 9801 40  0000 C CNN
+F 1 "R" V 11157 9801 40  0000 C CNN
 F 2 "~" V 11080 9800 30  0000 C CNN
 F 3 "~" H 11150 9800 30  0000 C CNN
@@
 P 12150 9200
 F 0 "Q4" H 12150 9050 60  0000 R CNN
-F 1 "MPSA92" V 12150 9700 60  0000 R CNN
+F 1 "MPSA92" V 12150 8900 60  0000 R CNN
 F 2 "~" H 12150 9200 60  0000 C CNN
 F 3 "~" H 12150 9200 60  0000 C CNN
 	1    12150 9200
-	1    0    0    -1
+	1    0    0    1
 $EndComp
 $Comp
@@
 P 12250 9800
 F 0 "R23" V 12330 9800 40  0000 C CNN
-F 1 "8k2" V 12257 9801 40  0000 C CNN
+F 1 "R" V 12257 9801 40  0000 C CNN
 F 2 "~" V 12180 9800 30  0000 C CNN
 F 3 "~" H 12250 9800 30  0000 C CNN
@@
 P 13250 9200
 F 0 "Q5" H 13250 9050 60  0000 R CNN
-F 1 "MPSA92" V 13250 9700 60  0000 R CNN
+F 1 "MPSA92" V 13250 8900 60  0000 R CNN
 F 2 "~" H 13250 9200 60  0000 C CNN
 F 3 "~" H 13250 9200 60  0000 C CNN
 	1    13250 9200
-	1    0    0    -1
+	1    0    0    1
 $EndComp
 $Comp
@@
 P 13350 9800
 F 0 "R24" V 13430 9800 40  0000 C CNN
-F 1 "8k2" V 13357 9801 40  0000 C CNN
+F 1 "R" V 13357 9801 40  0000 C CNN
 F 2 "~" V 13280 9800 30  0000 C CNN
 F 3 "~" H 13350 9800 30  0000 C CNN
@@
 P 14350 9200
 F 0 "Q6" H 14350 9050 60  0000 R CNN
-F 1 "MPSA92" V 14350 9700 60  0000 R CNN
+F 1 "MPSA92" V 14350 8900 60  0000 R CNN
 F 2 "~" H 14350 9200 60  0000 C CNN
 F 3 "~" H 14350 9200 60  0000 C CNN
 	1    14350 9200
-	1    0    0    -1
+	1    0    0    1
 $EndComp
 $Comp
@@
 P 14450 9800
 F 0 "R25" V 14530 9800 40  0000 C CNN
-F 1 "8k2" V 14457 9801 40  0000 C CNN
+F 1 "R" V 14457 9801 40  0000 C CNN
 F 2 "~" V 14380 9800 30  0000 C CNN
 F 3 "~" H 14450 9800 30  0000 C CNN
@@
 P 15450 9200
 F 0 "Q7" H 15450 9050 60  0000 R CNN
-F 1 "MPSA92" V 15450 9700 60  0000 R CNN
+F 1 "MPSA92" V 15450 8900 60  0000 R CNN
 F 2 "~" H 15450 9200 60  0000 C CNN
 F 3 "~" H 15450 9200 60  0000 C CNN
 	1    15450 9200
-	1    0    0    -1
+	1    0    0    1
 $EndComp
 $Comp
@@
 P 15550 9800
 F 0 "R26" V 15630 9800 40  0000 C CNN
-F 1 "8k2" V 15557 9801 40  0000 C CNN
+F 1 "R" V 15557 9801 40  0000 C CNN
 F 2 "~" V 15480 9800 30  0000 C CNN
 F 3 "~" H 15550 9800 30  0000 C CNN
@@
 Text Label 13350 1600 0    60   ~ 0
 GND
-Text Label 5150 3700 2    60   ~ 0
+Text Label 4900 3400 2    60   ~ 0
 GND
 Text Label 6150 8750 2    60   ~ 0
@@
 Wire Wire Line
 	2750 4550 2550 4550
+Text Label 2550 4750 2    60   ~ 0
+TXD
+Wire Wire Line
+	2750 4750 2550 4750
 Text Label 2550 4550 2    60   ~ 0
-TXD
-Wire Wire Line
-	2750 4750 2550 4750
-Text Label 2550 4750 2    60   ~ 0
 RXD
 $Comp
@@
 Wire Wire Line
 	6950 6000 6950 6300
+Text Label 5700 1950 2    60   ~ 0
+BUZ+
+Text Label 5700 2250 2    60   ~ 0
+BUZ-
+$Comp
+L R R5
+U 1 1 54EC1E92
+P 5100 2950
+F 0 "R5" V 5180 2950 40  0000 C CNN
+F 1 "10k" V 5107 2951 40  0000 C CNN
+F 2 "~" V 5030 2950 30  0000 C CNN
+F 3 "~" H 5100 2950 30  0000 C CNN
+	1    5100 2950
+	1    0    0    -1
+$EndComp
+Wire Wire Line
+	5100 2550 5100 2700
+Connection ~ 5100 2550
+Wire Wire Line
+	5100 3200 5100 3400
+Connection ~ 5100 3400
+Text Notes 14150 800  0    60   ~ 0
+REVISION NOTES V2 2015-03-19\n(A) R21-R26 WERE 8K2
+Text Notes 9850 9850 0    60   ~ 0
+(A)
 $EndSCHEMATC

Commit message: More Board Edits
Other:
- note added: "(B)"
- note added: "REVISION NOTES V2.1 2015-04-05\n(B) BIT0-3 LABELS INVERTED.\n CIRCUIT UNCHANGED."
- moved on the sheet: P1
Changed lines of the file:
@@
 Sheet 1 2
 Title "NIXIEBOARD"
-Date "18 mar 2015"
+Date "5 apr 2015"
 Rev "V2"
 Comp ""
@@
 	1    0    0    -1
 $EndComp
-Text Label 13350 1400 0    60   ~ 0
+Text Label 11200 2650 0    60   ~ 0
 VSUP
 Text Label 2200 9600 2    60   ~ 0
@@
 S3
 Text Label 3450 3800 0    60   ~ 0
+BIT0
+Text Label 3450 3700 0    60   ~ 0
+BIT1
+Text Label 3450 3600 0    60   ~ 0
+BIT2
+Text Label 3450 3500 0    60   ~ 0
 BIT3
-Text Label 3450 3700 0    60   ~ 0
-BIT2
-Text Label 3450 3600 0    60   ~ 0
-BIT1
-Text Label 3450 3500 0    60   ~ 0
-BIT0
 Text Label 2950 6000 2    60   ~ 0
 MISO
@@
 $EndComp
 Text Label 2200 9800 2    60   ~ 0
+BIT2
+Text Label 2200 9700 2    60   ~ 0
 BIT1
-Text Label 2200 9700 2    60   ~ 0
-BIT2
 Text Label 2200 9400 2    60   ~ 0
+BIT0
+Text Label 2200 9500 2    60   ~ 0
 BIT3
-Text Label 2200 9500 2    60   ~ 0
-BIT0
 $Comp
 L K155ID1 U2
@@
 L CONN_2 P1
 U 1 1 54AF9004
-P 12700 1500
-F 0 "P1" V 12650 1500 40  0000 C CNN
-F 1 "PWR" V 12750 1500 40  0000 C CNN
-F 2 "" H 12700 1500 60  0000 C CNN
-F 3 "" H 12700 1500 60  0000 C CNN
-	1    12700 1500
+P 10550 2750
+F 0 "P1" V 10500 2750 40  0000 C CNN
+F 1 "PWR" V 10600 2750 40  0000 C CNN
+F 2 "" H 10550 2750 60  0000 C CNN
+F 3 "" H 10550 2750 60  0000 C CNN
+	1    10550 2750
 	-1   0    0    1
 $EndComp
@@
 GND
 Wire Wire Line
-	13350 1400 13050 1400
-Wire Wire Line
-	13050 1600 13350 1600
-Text Notes 12700 1200 0    60   ~ 0
+	11200 2650 10900 2650
+Wire Wire Line
+	10900 2850 11200 2850
+Text Notes 10550 2450 0    60   ~ 0
 POWER INPUT
 Text Notes 12300 4300 0    60   ~ 0
@@
 Text Label 3000 8800 0    60   ~ 0
 GND
-Text Label 13350 1600 0    60   ~ 0
+Text Label 11200 2850 0    60   ~ 0
 GND
 Text Label 4900 3400 2    60   ~ 0
@@
 	5100 3200 5100 3400
 Connection ~ 5100 3400
-Text Notes 14150 800  0    60   ~ 0
+Text Notes 14250 800  0    60   ~ 0
 REVISION NOTES V2 2015-03-19\n(A) R21-R26 WERE 8K2
 Text Notes 9850 9850 0    60   ~ 0
 (A)
+Text Notes 14250 1100 0    60   ~ 0
+REVISION NOTES V2.1 2015-04-05\n(B) BIT0-3 LABELS INVERTED.\n         CIRCUIT UNCHANGED.
+Text Notes 3700 3650 0    60   ~ 0
+(B)
+Text Notes 1800 9600 0    60   ~ 0
+(B)
 $EndSCHEMATC

Commit message: Add board design
Parts:
- C1, C2, C3, C6, C7: symbol C -> Device:C
- C4, C5: symbol CP1 -> Device:CP1
- D1: symbol ZENER -> nixieclockboard-rescue:ZENER
- IC1: symbol ATMEGA328P-A -> nixieclockboard-rescue:ATMEGA328P-A
- JP1, JP2, JP3: symbol JUMPER3 -> nixieclockboard-rescue:JUMPER3
- P1, P11, P12, P13, P2, P4, P7, P8: symbol CONN_2 -> nixieclockboard-rescue:CONN_2
- P10: symbol CONN_6 -> nixieclockboard-rescue:CONN_6
- P5: symbol CONN_4 -> nixieclockboard-rescue:CONN_4
- P6: symbol AVRISP6 -> nixieclockboard-rescue:AVRISP6
- P9: symbol CONN_12 -> nixieclockboard-rescue:CONN_12
- Q1: symbol MOSFET_N -> nixieclockboard-rescue:MOSFET_N
- Q10, Q11, Q12, Q13, Q14, Q15, Q8, Q9: symbol NPN -> nixieclockboard-rescue:NPN
- Q2, Q3, Q4, Q5, Q6, Q7: symbol PNP -> nixieclockboard-rescue:PNP
- R1, R10, R11, R12, R13, R14, R15, R16, R17, R18, R19, R2, R20, R21, R22, R23, R24, R25, R26, R27, R28, R29, R3, R30, R31, R32, R4, R5, R6, R7, R8, R9: symbol R -> Device:R
- U1: symbol LM1117 -> nixieclockboard-rescue:LM1117
- U2: symbol K155ID1 -> nixieclockboard-rescue:K155ID1
- X1: symbol CRYSTAL -> nixieclockboard-rescue:CRYSTAL
Connections:
- wire segments 225 -> 274
Other:
- note added: "REVISION NOTES 03 2017-10-03\n(C) UPDATE TO NEW SYMBOL LIBRARIES"
