File: board/nixieclockboard_hvsupply.sch (KiCad schematic (older format))
At the start: 16 parts

Commit message: Schematic and board creation continued
Parts:
- gave numbers to parts that had none: 16
Changed lines of the file:
@@
 $Descr A4 11693 8268
 encoding utf-8
-Sheet 2 8
+Sheet 2 2
 Title ""
-Date "11 jan 2015"
+Date "21 jan 2015"
 Rev ""
 Comp ""
@@
 VPUMP
 $Comp
-L CP1 C?
+L CP1 C9
 U 1 1 4DE4DB6D
 P 1950 3000
-F 0 "C?" H 2000 3100 50  0000 L CNN
+F 0 "C9" H 2000 3100 50  0000 L CNN
 F 1 "10u" H 2000 2900 50  0000 L CNN
 F 2 "" H 1950 3000 60  0001 C CNN
@@
 $EndComp
 $Comp
-L C C?
+L C C10
 U 1 1 4DE4C610
 P 2500 3750
-F 0 "C?" H 2550 3850 50  0000 L CNN
+F 0 "C10" H 2550 3850 50  0000 L CNN
 F 1 "100p" H 2550 3650 50  0000 L CNN
 F 2 "" H 2500 3750 60  0001 C CNN
@@
 $EndComp
 $Comp
-L R R?
+L R R37
 U 1 1 4DE4C60C
 P 2500 3200
-F 0 "R?" V 2580 3200 50  0000 C CNN
+F 0 "R37" V 2580 3200 50  0000 C CNN
 F 1 "2k2" V 2500 3200 50  0000 C CNN
 F 2 "" H 2500 3200 60  0001 C CNN
@@
 $EndComp
 $Comp
-L MOSFET_N Q?
+L MOSFET_N Q16
 U 1 1 4DE4C5DB
 P 3050 2900
-F 0 "Q?" H 3060 3070 60  0000 R CNN
+F 0 "Q16" H 3060 3070 60  0000 R CNN
 F 1 "IRF740" H 3060 2750 60  0000 R CNN
 F 2 "" H 3050 2900 60  0001 C CNN
@@
 VOUT
 $Comp
-L DIODE D?
+L DIODE D2
 U 1 1 4DE4C58A
 P 2450 2050
-F 0 "D?" H 2450 2150 40  0000 C CNN
+F 0 "D2" H 2450 2150 40  0000 C CNN
 F 1 "UF4004" H 2450 1950 40  0000 C CNN
 F 2 "" H 2450 2050 60  0001 C CNN
@@
 $EndComp
 $Comp
-L INDUCTOR L?
+L INDUCTOR L1
 U 1 1 4DE4C57D
 P 4350 2050
-F 0 "L?" V 4300 2050 40  0000 C CNN
+F 0 "L1" V 4300 2050 40  0000 C CNN
 F 1 "100uH" V 4450 2050 40  0000 C CNN
 F 2 "" H 4350 2050 60  0001 C CNN
@@
 $EndComp
 $Comp
-L CP1 C?
+L CP1 C8
 U 1 1 4DE4C547
 P 6150 2850
-F 0 "C?" H 6200 2950 50  0000 L CNN
+F 0 "C8" H 6200 2950 50  0000 L CNN
 F 1 "330u" H 6200 2750 50  0000 L CNN
 F 2 "" H 6150 2850 60  0001 C CNN
@@
 $EndComp
 $Comp
-L C C?
+L C C11
 U 1 1 4DE4C52B
 P 5050 4050
-F 0 "C?" H 5100 4150 50  0000 L CNN
+F 0 "C11" H 5100 4150 50  0000 L CNN
 F 1 "2n2" H 5100 3950 50  0000 L CNN
 F 2 "" H 5050 4050 60  0001 C CNN
@@
 $EndComp
 $Comp
-L R R?
+L R R38
 U 1 1 4DE4C4E1
 P 1300 4050
-F 0 "R?" V 1380 4050 50  0000 C CNN
+F 0 "R38" V 1380 4050 50  0000 C CNN
 F 1 "470" V 1300 4050 50  0000 C CNN
 F 2 "" H 1300 4050 60  0001 C CNN
@@
 $EndComp
 $Comp
-L POT RV?
+L POT RV1
 U 1 1 4DE4C4DD
 P 1300 3450
-F 0 "RV?" H 1300 3350 50  0000 C CNN
+F 0 "RV1" H 1300 3350 50  0000 C CNN
 F 1 "1k" H 1300 3450 50  0000 C CNN
 F 2 "" H 1300 3450 60  0001 C CNN
@@
 $EndComp
 $Comp
-L R R?
+L R R35
 U 1 1 4DE4C4D7
 P 1300 2850
-F 0 "R?" V 1380 2850 50  0000 C CNN
+F 0 "R35" V 1380 2850 50  0000 C CNN
 F 1 "220k" V 1300 2850 50  0000 C CNN
 F 2 "" H 1300 2850 60  0001 C CNN
@@
 $EndComp
 $Comp
-L NPN Q?
+L NPN Q17
 U 1 1 4DE4C4AF
 P 5650 3900
-F 0 "Q?" H 5650 3750 50  0000 R CNN
+F 0 "Q17" H 5650 3750 50  0000 R CNN
 F 1 "BC547" H 5650 4050 50  0000 R CNN
 F 2 "" H 5650 3900 60  0001 C CNN
@@
 $EndComp
 $Comp
-L R R?
+L R R34
 U 1 1 4DE4C492
 P 5750 2450
-F 0 "R?" V 5830 2450 50  0000 C CNN
+F 0 "R34" V 5830 2450 50  0000 C CNN
 F 1 "56k" V 5750 2450 50  0000 C CNN
 F 2 "" H 5750 2450 60  0001 C CNN
@@
 $EndComp
 $Comp
-L R R?
+L R R36
 U 1 1 4DE4C448
 P 5450 3150
-F 0 "R?" V 5530 3150 50  0000 C CNN
+F 0 "R36" V 5530 3150 50  0000 C CNN
 F 1 "10k" V 5450 3150 50  0000 C CNN
 F 2 "" H 5450 3150 60  0001 C CNN
@@
 $EndComp
 $Comp
-L R R?
+L R R33
 U 1 1 4DE4C442
 P 5450 2450
-F 0 "R?" V 5530 2450 50  0000 C CNN
+F 0 "R33" V 5530 2450 50  0000 C CNN
 F 1 "1k" V 5450 2450 50  0000 C CNN
 F 2 "" H 5450 2450 60  0001 C CNN
@@
 $EndComp
 $Comp
-L 555 U?
+L 555 U3
 U 1 1 4DE4C405
 P 3750 3200
-F 0 "U?" H 4350 3850 60  0000 C CNN
+F 0 "U3" H 4350 3850 60  0000 C CNN
 F 1 "555" H 4350 3250 60  0000 C CNN
 F 2 "" H 3750 3200 60  0001 C CNN
@@
 	1    0    0    -1
 $EndComp
+Text HLabel 5150 1850 1    60   Input ~ 0
+VIN
 Text GLabel 1150 4350 0    60   Input ~ 0
 GND
-Text HLabel 5150 1850 1    60   Input ~ 0
-VIN
 $EndSCHEMATC

Commit message: Board completed
Changed lines of the file:
@@
 encoding utf-8
 Sheet 2 2
-Title ""
-Date "21 jan 2015"
-Rev ""
+Title "NIXIEBOARD"
+Date "18 mar 2015"
+Rev "V2"
 Comp ""
 Comment1 ""
@@
 	2500 3950 2500 4350
 Connection ~ 2500 4350
-Wire Wire Line
-	1950 2800 1950 2050
 Connection ~ 1950 2050
 Text Label 1300 3750 0    60   ~ 0
@@
 Text GLabel 1150 4350 0    60   Input ~ 0
 GND
+Wire Wire Line
+	1950 2050 1950 2800
 $EndSCHEMATC

Commit message: Add board design
Parts:
- C10, C11: symbol C -> Device:C
- C8, C9: symbol CP1 -> Device:CP1
- D2: symbol DIODE -> nixieclockboard-rescue:DIODE
- L1: symbol INDUCTOR -> nixieclockboard-rescue:INDUCTOR
- Q16: symbol MOSFET_N -> nixieclockboard-rescue:MOSFET_N
- Q17: symbol NPN -> nixieclockboard-rescue:NPN
- R33, R34, R35, R36, R37, R38: symbol R -> Device:R
- RV1: symbol POT -> nixieclockboard-rescue:POT
- U3: symbol 555 -> nixieclockboard-rescue:555
Other:
- note added: "REVISION NOTES 03 2017-10-03\n(A) UPDATED SYMBOLS TO NEW LIBRARY"
- moved on the sheet: RV1
